File: drone/drone.sch (KiCad schematic (older format))
At the start: 1 part

Commit message: new libraries
Parts:
- removed U?: ATmega328-AU, Package_QFP:TQFP-32_7x7mm_P0.8mm, symbol MCU_Microchip_ATmega:ATmega328-AU
- added U1: Pico, MCU_RaspberryPi_and_Boards:RPi_Pico_SMD_TH, symbol MCU_RaspberryPi_and_Boards:Pico
Connections:
- no-connect marks 0 -> 1
Changed lines of the file:
@@
 Comment4 ""
 $EndDescr
+NoConn ~ 8250 1600
 $Comp
-L MCU_Microchip_ATmega:ATmega328-AU U?
-U 1 1 6191BB19
-P 2300 3750
-F 0 "U?" H 2300 2161 50  0000 C CNN
-F 1 "ATmega328-AU" H 2300 2070 50  0000 C CNN
-F 2 "Package_QFP:TQFP-32_7x7mm_P0.8mm" H 2300 3750 50  0001 C CIN
-F 3 "http://ww1.microchip.com/downloads/en/DeviceDoc/ATmega328_P%20AVR%20MCU%20with%20picoPower%20Technology%20Data%20Sheet%2040001984A.pdf" H 2300 3750 50  0001 C CNN
-	1    2300 3750
+L MCU_RaspberryPi_and_Boards:Pico U1
+U 1 1 6191C1D5
+P 3400 2150
+F 0 "U1" H 3400 3365 50  0000 C CNN
+F 1 "Pico" H 3400 3274 50  0000 C CNN
+F 2 "MCU_RaspberryPi_and_Boards:RPi_Pico_SMD_TH" V 3400 2150 50  0001 C CNN
+F 3 "" H 3400 2150 50  0001 C CNN
+	1    3400 2150
 	1    0    0    -1
 $EndComp
